File: ruler.kicad_pcb (KiCad board)
At the start: 2 copper layers, 152.4 x 31.8 mm, 61 parts

Commit message: Update datestamp. Update gerbers and images
Other:
- board text added: "Max Proskauer Version 0.1 Dec 2021"
- board text removed: "Max Proskauer Version 0.1 Aug 2020"
Changed lines of the file:
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@@
       (drillshape 0)
       (scaleselection 1)
-      (outputdirectory "export/gerber"))
+      (outputdirectory "gerber"))
   )
   (net 0 "")
@@
     (effects (font (size 1.2 1.2) (thickness 0.2)) (justify mirror))
   )
-  (gr_text "Max Proskauer  Version 0.1  Aug 2020" (at 114.3 100.965) (layer B.Cu)
+  (gr_text "Max Proskauer  Version 0.1  Dec 2021" (at 114.3 100.965) (layer B.Cu)
     (effects (font (size 1 1) (thickness 0.2)) (justify mirror))
   )

Commit message: Update to KiCad 6.0
Other:
- net class Default removed
