File: ruler/ruler.kicad_pcb (KiCad board)
At the start: 2 copper layers, 152.4 x 31.8 mm, 61 parts

Commit message: Update timestamp. Regenerate gerbers
Other:
- rule pad_to_mask_clearance: 0.051 -> 0
- board text added: "Max Proskauer Version 0.1 May 2022"
- board text removed: "Max Proskauer Version 0.1 Dec 2021"
Changed lines of the file:
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@@
   )
   (setup
-    (pad_to_mask_clearance 0.051)
-    (solder_mask_min_width 0.25)
+    (stackup
+      (layer "F.SilkS" (type "Top Silk Screen"))
+      (layer "F.Paste" (type "Top Solder Paste"))
+      (layer "F.Mask" (type "Top Solder Mask") (thickness 0.01))
+      (layer "F.Cu" (type "copper") (thickness 0.035))
+      (layer "dielectric 1" (type "core") (thickness 1.51) (material "FR4") (epsilon_r 4.5) (loss_tangent 0.02))
+      (layer "B.Cu" (type "copper") (thickness 0.035))
+      (layer "B.Mask" (type "Bottom Solder Mask") (thickness 0.01))
+      (layer "B.Paste" (type "Bottom Solder Paste"))
+      (layer "B.SilkS" (type "Bottom Silk Screen"))
+      (copper_finish "None")
+      (dielectric_constraints no)
+    )
+    (pad_to_mask_clearance 0)
     (pcbplotparams
       (layerselection 0x00010f0_ffffffff)
@@
     (fp_line (start 3.15 1.6) (end -3.15 1.6) (layer "F.Fab") (width 0.1))
     (fp_line (start -3.15 1.6) (end -3.15 -1.6) (layer "F.Fab") (width 0.1))
-    (pad "1" smd roundrect locked (at -2.9 0) (size 1.35 3.35) (layers "F.Cu" "F.Paste" "F.Mask") (roundrect_rratio 0.185185))
-    (pad "2" smd roundrect locked (at 2.9 0) (size 1.35 3.35) (layers "F.Cu" "F.Paste" "F.Mask") (roundrect_rratio 0.185185))
+    (pad "1" smd roundrect locked (at -2.9 0) (size 1.35 3.35) (layers "F.Cu" "F.Paste" "F.Mask") (roundrect_rratio 0.1851851852))
+    (pad "2" smd roundrect locked (at 2.9 0) (size 1.35 3.35) (layers "F.Cu" "F.Paste" "F.Mask") (roundrect_rratio 0.1851851852))
     (model "${KISYS3DMOD}/Resistor_SMD.3dshapes/R_2512_6332Metric.wrl"
       (offset (xyz 0 0 0))
@@
     (fp_line (start 2.25 -0.8) (end 2.25 0.8) (layer "F.Fab") (width 0.1))
     (fp_line (start 2.25 0.8) (end -2.25 0.8) (layer "F.Fab") (width 0.1))
-    (pad "1" smd roundrect locked (at -2 0) (size 1.4 1.8) (layers "F.Cu" "F.Paste" "F.Mask") (roundrect_rratio 0.178571))
-    (pad "2" smd roundrect locked (at 2 0) (size 1.4 1.8) (layers "F.Cu" "F.Paste" "F.Mask") (roundrect_rratio 0.178571))
+    (pad "1" smd roundrect locked (at -2 0) (size 1.4 1.8) (layers "F.Cu" "F.Paste" "F.Mask") (roundrect_rratio 0.1785707143))
+    (pad "2" smd roundrect locked (at 2 0) (size 1.4 1.8) (layers "F.Cu" "F.Paste" "F.Mask") (roundrect_rratio 0.1785707143))
     (model "${KISYS3DMOD}/Resistor_SMD.3dshapes/R_1806_4516Metric.wrl"
       (offset (xyz 0 0 0))
@@
     (fp_line (start -2.5 -1.25) (end 2.5 -1.25) (layer "F.Fab") (width 0.1))
     (fp_line (start 2.5 -1.25) (end 2.5 1.25) (layer "F.Fab") (width 0.1))
-    (pad "1" smd roundrect locked (at -2.25 0) (size 1.35 2.65) (layers "F.Cu" "F.Paste" "F.Mask") (roundrect_rratio 0.185185))
-    (pad "2" smd roundrect locked (at 2.25 0) (size 1.35 2.65) (layers "F.Cu" "F.Paste" "F.Mask") (roundrect_rratio 0.185185))
+    (pad "1" smd roundrect locked (at -2.25 0) (size 1.35 2.65) (layers "F.Cu" "F.Paste" "F.Mask") (roundrect_rratio 0.1851851852))
+    (pad "2" smd roundrect locked (at 2.25 0) (size 1.35 2.65) (layers "F.Cu" "F.Paste" "F.Mask") (roundrect_rratio 0.1851851852))
     (model "${KISYS3DMOD}/Resistor_SMD.3dshapes/R_2010_5025Metric.wrl"
       (offset (xyz 0 0 0))
@@
     (effects (font (size 1.2 1.2) (thickness 0.2) italic) (justify right))
   )
-  (gr_text "Max Proskauer  Version 0.1  Dec 2021" (at 114.3 100.965) (layer "B.Cu")
+  (gr_text "Max Proskauer  Version 0.1  May 2022" (at 114.3 100.965) (layer "B.Cu")
     (effects (font (size 1 1) (thickness 0.2)) (justify mirror))
   )
